File: tests/fixtures/testproj.kicad_sch (KiCad schematic)
At the start: 2 parts, among them U3 F0D3180

Commit message: Auto-apply built-in sim models and improve datasheet discovery
Write KiCad simulation fields for standard passives, diodes, and batteries
on context refresh so parts like 1N4007 no longer need manual Simulation
Model setup. Enable spice_write_symbol_fields by default and extend gap
detection to all sim-participating symbols.

Improve AI datasheet discovery with per-URL attempt logging, OnSemi direct-PDF
heuristics, portal URL filtering, and a richer missing-datasheets UI for
reviewing failures and approving downloads. Add launcher dialog entry point,
netlist export hardening, and tests/docs for the new flows.
Parts:
- R1: Spice_Model (none) -> 10k; Spice_Primitive (none) -> R
Changed lines of the file:
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@@
       (at 100 110 0)
+    )
+    (property "Sim.Params" "r=10k"
+      (at 0 0 0)
+    )
+    (property "Sim.Pins" "1=1 2=2"
+      (at 0 0 0)
+    )
+    (property "Sim.Type" "RESISTOR"
+      (at 0 0 0)
+    )
+    (property "Sim.Device" "R"
+      (at 0 0 0)
+    )
+    (property "Spice_Primitive" "R"
+      (at 0 0 0)
+    )
+    (property "Spice_Model" "10k"
+      (at 0 0 0)
     )
     (property "Footprint" "Resistor_SMD:R_0805"
